Commit message: Gazebo sim and control added

File: description/robot_core.xacro (robot description, xacro)
@@ -39,4 +39,7 @@
         </xacro:inertial_box>
     </link>
+    <gazebo reference="chassis">
+        <material>Gazebo/White</material>
+    </gazebo>
     <joint name="left_front_wheel_joint" type = "continuous">
         <parent link = "base_link"/>
@@ -61,4 +64,9 @@
         </xacro:inertial_cylinder>
     </link>
+    <gazebo reference="left_front_wheel">
+        <material>Gazebo/Blue</material>
+        <mu1 value = "0.001"/>
+        <mu2 value = "0.001"/>
+    </gazebo>
     <joint name="right_front_wheel_joint" type = "continuous">
         <parent link = "base_link"/>
@@ -83,4 +91,9 @@
         </xacro:inertial_cylinder>
     </link>
+    <gazebo reference="right_front_wheel">
+        <material>Gazebo/Blue</material>
+        <mu1 value = "0.001"/>
+        <mu2 value = "0.001"/>
+    </gazebo>
     <joint name="left_back_wheel_joint" type = "continuous">
         <parent link = "base_link"/>
@@ -105,4 +118,7 @@
         </xacro:inertial_cylinder>
     </link>
+    <gazebo reference="left_back_wheel">
+        <material>Gazebo/Blue</material>
+    </gazebo>
     <joint name="right_back_wheel_joint" type = "continuous">
         <parent link = "base_link"/>
@@ -127,3 +143,6 @@
         </xacro:inertial_cylinder>
     </link>
+    <gazebo reference="right_back_wheel">
+        <material>Gazebo/Blue</material>
+    </gazebo>
 </robot>

Commit message: Added LIDAR sensing in simulation

File: description/robot_core.xacro (robot description, xacro)
@@ -13,4 +13,7 @@
     <material name = "black" >
         <color rgba = "0 0 0 1"/>
+    </material>
+    <material name = "red" >
+        <color rgba = "1 0 0 1"/>
     </material>
     <link name = "base_link">
@@ -42,5 +45,5 @@
         <material>Gazebo/White</material>
     </gazebo>
-    <joint name="left_front_wheel_joint" type = "continuous">
+    <joint name="left_front_wheel_joint" type = "fixed">
         <parent link = "base_link"/>
         <child link = "left_front_wheel"/>
@@ -69,5 +72,5 @@
         <mu2 value = "0.001"/>
     </gazebo>
-    <joint name="right_front_wheel_joint" type = "continuous">
+    <joint name="right_front_wheel_joint" type = "fixed">
         <parent link = "base_link"/>
         <child link = "right_front_wheel"/>
