Commit message: Twist mux and nav2 implemented. Need to add params files to repo

File: description/lidar.xacro (robot description, xacro)
@@ -25,5 +25,5 @@
         <sensor name="laser" type = "ray">
             <pose>0 0 0 0</pose>
-            <visualize>true</visualize>
+            <visualize>false</visualize>
             <update_rate>10</update_rate>
             <ray>

File: description/robot.urdf.xacro (robot description, xacro)
@@ -5,3 +5,4 @@
     <xacro:include filename="ros2_control.xacro"/>
     <xacro:include filename="lidar.xacro"/>
+    <xacro:include filename="camera.xacro"/>
 </robot>

File: description/robot_core.xacro (robot description, xacro)
@@ -18,4 +18,11 @@
     </material>
     <link name = "base_link">
+    </link>
+    <joint name = "base_footprint" type="fixed">
+        <parent link = "base_link"/>
+        <child link = "base_footprint"/>
+        <origin xyz = "0 0 0"/>
+    </joint>
+    <link name = "base_footprint">
     </link>
     <joint name = "chassis_joint" type="fixed">
